File: hw/business_card/business_card.kicad_sch (KiCad schematic)
At the start: 0 parts

Commit message: BoM complete
Other:
- company: (none) -> Adam Hagengruber
- title: (none) -> Business Card
Changed lines of the file:
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@@
 	(generator_version "10.0")
 	(paper "A4")
-	(sheet
-		(at 204.47 106.68)
+	(title_block
+		(title "Business Card")
+		(date "2026-10-06")
+		(rev "A")
+		(company "Adam Hagengruber")
+	)
+	(bezier
+		(pts
+			(xy 218.44 60.325) (xy 218.44 60.325) (xy 215.9 57.15) (xy 215.9 57.15)
+		)
+		(stroke
+			(width 0.254)
+			(type solid)
+		)
+		(fill
+			(type none)
+		)
+	)
+	(bezier
+		(pts
+			(xy 170.18 69.85) (xy 170.18 69.85) (xy 166.37 66.04) (xy 166.37 66.04)
+		)
+		(stroke
+			(width 0.254)
+			(type solid)
+		)
+		(fill
+			(type none)
+		)
+	)
+	(bezier
+		(pts
+			(xy 95.25 95.25) (xy 95.25 95.25) (xy 98.425 92.075) (xy 98.425 92.075)
+		)
+		(stroke
+			(width 0.254)
+			(type solid)
+		)
+		(fill
+			(type none)
+		)
+	)
+	(bezier
+		(pts
+			(xy 98.425 92.075) (xy 95.25 88.9) (xy 95.25 88.9) (xy 95.25 88.9)
+		)
+		(stroke
+			(width 0.254)
+			(type solid)
+		)
+		(fill
+			(type none)
+		)
+	)
+	(bezier
+		(pts
+			(xy 166.37 73.66) (xy 166.37 73.66) (xy 170.18 69.85) (xy 170.18 69.85)
+		)
+		(stroke
+			(width 0.254)
+			(type solid)
+		)
+		(fill
+			(type none)
+		)
+	)
+	(bezier
+		(pts
+			(xy 218.44 60.325) (xy 218.44 60.325) (xy 215.9 63.5) (xy 215.9 63.5)
+		)
+		(stroke
+			(width 0.254)
+			(type solid)
+		)
+		(fill
+			(type none)
+		)
+	)
+	(polyline
+		(pts
+			(xy 208.915 60.325) (xy 218.44 60.325)
+		)
+		(stroke
+			(width 0.254)
+			(type solid)
+		)
+	)
+	(polyline
+		(pts
+			(xy 157.48 69.85) (xy 170.18 69.85)
+		)
+		(stroke
+			(width 0.254)
+			(type solid)
+		)
+	)
+	(polyline
+		(pts
+			(xy 68.58 92.075) (xy 98.425 92.075)
+		)
+		(stroke
+			(width 0.254)
+			(type solid)
+		)
+	)
+	(sheet
+		(at 218.44 48.26)
 		(size 26.67 25.4)
 		(exclude_from_sim no)
@@
 		)
 		(property "Sheetname" "Display"
-			(at 204.47 105.9684 0)
+			(at 218.44 47.5484 0)
 			(show_name no)
 			(do_not_autoplace no)
@@
 		)
 		(property "Sheetfile" "display.kicad_sch"
-			(at 204.47 132.6646 0)
+			(at 218.44 74.2446 0)
 			(show_name no)
 			(do_not_autoplace no)
@@
 	)
 	(sheet
-		(at 169.418 35.814)
+		(at 170.053 44.069)
 		(size 38.608 32.258)
 		(exclude_from_sim no)
@@
 		)
 		(property "Sheetname" "Display Driver"
-			(at 169.418 35.1024 0)
+			(at 170.053 43.3574 0)
 			(show_name no)
 			(do_not_autoplace no)
@@
 		)
 		(property "Sheetfile" "display_driver.kicad_sch"
-			(at 169.418 68.6566 0)
+			(at 170.053 76.9116 0)
 			(show_name no)
 			(do_not_autoplace no)
@@
 	)
 	(sheet
-		(at 129.54 81.28)
-		(size 38.1 27.94)
+		(at 98.425 66.04)
+		(size 59.055 52.705)
 		(exclude_from_sim no)
 		(in_bom yes)
@@
 		)
 		(property "Sheetname" "MCU"
-			(at 129.54 80.5684 0)
+			(at 98.425 65.3284 0)
 			(show_name no)
 			(do_not_autoplace no)
@@
 		)
 		(property "Sheetfile" "mcu.kicad_sch"
-			(at 129.54 109.8046 0)
+			(at 98.425 119.3296 0)
 			(show_name no)
 			(do_not_autoplace no)
@@
 	)
 	(sheet
-		(at 24.384 24.892)
+		(at 28.194 79.502)
 		(size 40.386 27.686)
 		(exclude_from_sim no)
@@
 		)
 		(property "Sheetname" "Power Input"
-			(at 24.384 24.1804 0)
+			(at 28.194 78.7904 0)
 			(show_name no)
 			(do_not_autoplace no)
@@
 		)
 		(property "Sheetfile" "power_input.kicad_sch"
-			(at 24.384 53.1626 0)
-			(show_name no)
-			(do_not_autoplace no)
+			(at 28.194 107.7726 0)
+			(show_name no)
+			(do_not_autoplace no)
