File: hw/business_card/display.kicad_sch (KiCad schematic)
At the start: 36 parts

Commit message: BoM complete
Other:
- title: (none) -> Display
Changed lines of the file:
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@@
 	(generator_version "10.0")
 	(paper "A4")
+	(title_block
+		(title "Display")
+		(date "2026-10-06")
+		(rev "A")
+	)
 	(rectangle
 		(start 43.18 26.67)
