File: hw/business_card/display_driver.kicad_sch (KiCad schematic)
At the start: 12 parts, among them U3 PCAL6416AHF_128, U4 PCAL6416AHF_128

Commit message: BoM complete
Other:
- title: (none) -> Display Driver
Changed lines of the file:
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@@
 	(generator_version "10.0")
 	(paper "A4")
+	(title_block
+		(title "Display Driver")
+		(date "2026-10-06")
+		(rev "A")
+	)
 	(rectangle
 		(start 172.72 102.87)
