File: hw/business_card/mcu.kicad_sch (KiCad schematic)
At the start: 40 parts, among them J2 Conn_01x02_Pin, Q2 2N7002NXAKR, Q3 2N7002NXAKR, SW1 3983, SW2 3983, U1 PIC16F15245T-I/REB, U5 LM8365BALMF27/NOPB, U6 TMP1075NDRLR

Commit message: BoM complete
Parts:
- TP1, TP2, TP3, TP4, TP5: footprint (none) -> TestPoint:TestPoint_Pad_D2.5mm
Other:
- title: (none) -> MCU and Logic
Changed lines of the file:
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@@
 	(generator_version "10.0")
 	(paper "A4")
+	(title_block
+		(title "MCU and Logic")
+		(date "2026-10-06")
+		(rev "A")
+	)
 	(rectangle
 		(start 28.829 27.178)
@@
 			)
 		)
-		(property "Footprint" ""
+		(property "Footprint" "TestPoint:TestPoint_Pad_D2.5mm"
 			(at 262.89 53.34 0)
 			(hide yes)
@@
 			)
 		)
-		(property "Footprint" ""
+		(property "Footprint" "TestPoint:TestPoint_Pad_D2.5mm"
 			(at 262.89 58.42 0)
 			(hide yes)
@@
 			)
 		)
-		(property "Footprint" ""
+		(property "Footprint" "TestPoint:TestPoint_Pad_D2.5mm"
 			(at 262.89 63.5 0)
 			(hide yes)
@@
 			)
 		)
-		(property "Footprint" ""
+		(property "Footprint" "TestPoint:TestPoint_Pad_D2.5mm"
 			(at 262.89 43.18 0)
 			(hide yes)
@@
 			)
 		)
-		(property "Footprint" ""
+		(property "Footprint" "TestPoint:TestPoint_Pad_D2.5mm"
 			(at 262.89 48.26 0)
 			(hide yes)
