File: hw/business_card/power_input.kicad_sch (KiCad schematic)
At the start: 27 parts, among them J1 10164359-00011LF, Q1 2N7002NXAKR, U2 MCP7940MT-I/MNY, U7 LMV331IDBVRG4, Y1 ECS-327MVATX-2-CN-TR3

Commit message: BoM complete
Connections:
- net +5V: now also R51.1
- net GND: no longer R51.2
- net at Q1.1 (G), U7.4 (OUT): now also R51.2; no longer R51.1
Other:
- title: (none) -> Power Input
- moved on the sheet: R51
Changed lines of the file:
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@@
 	(generator_version "10.0")
 	(paper "A4")
+	(title_block
+		(title "Power Input")
+		(date "2026-10-06")
+		(rev "A")
+	)
 	(rectangle
 		(start 62.865 21.59)
@@
 	)
 	(junction
-		(at 125.73 182.88)
-		(diameter 0)
-		(color 0 0 0 0)
-	)
-	(junction
 		(at 30.48 165.1)
 		(diameter 0)
@@
 	)
 	(junction
-		(at 125.73 167.64)
+		(at 146.05 41.91)
 		(diameter 0)
 		(color 0 0 0 0)
 	)
 	(junction
-		(at 146.05 41.91)
+		(at 115.57 156.21)
 		(diameter 0)
 		(color 0 0 0 0)
@@
 	)
 	(junction
+		(at 124.46 167.64)
+		(diameter 0)
+		(color 0 0 0 0)
+	)
+	(junction
 		(at 68.58 91.44)
 		(diameter 0)
@@
 	(wire
 		(pts
-			(xy 101.6 167.64) (xy 125.73 167.64)
+			(xy 101.6 167.64) (xy 124.46 167.64)
 		)
 		(stroke
@@
 	(wire
 		(pts
+			(xy 115.57 156.21) (xy 115.57 165.1)
+		)
+		(stroke
+			(width 0)
+			(type default)
+		)
+	)
+	(wire
+		(pts
 			(xy 68.58 96.52) (xy 68.58 99.06)
 		)
@@
 	(wire
 		(pts
-			(xy 125.73 182.88) (xy 115.57 182.88)
+			(xy 115.57 182.88) (xy 143.51 182.88)
 		)
 		(stroke
@@
 	(wire
 		(pts
+			(xy 124.46 166.37) (xy 124.46 167.64)
+		)
+		(stroke
+			(width 0)
+			(type default)
+		)
+	)
+	(wire
+		(pts
 			(xy 67.31 55.88) (xy 67.31 57.15)
 		)
@@
 	(wire
 		(pts
-			(xy 125.73 167.64) (xy 130.81 167.64)
-		)
-		(stroke
-			(width 0)
-			(type default)
-		)
-	)
-	(wire
-		(pts
 			(xy 191.77 86.36) (xy 191.77 93.98)
 		)
@@
 	(wire
 		(pts
-			(xy 143.51 182.88) (xy 125.73 182.88)
+			(xy 20.32 180.34) (xy 30.48 180.34)
 		)
 		(stroke
@@
 	(wire
 		(pts
-			(xy 20.32 180.34) (xy 30.48 180.34)
+			(xy 133.35 41.91) (xy 133.35 45.72)
 		)
 		(stroke
@@
 	(wire
 		(pts
-			(xy 133.35 41.91) (xy 133.35 45.72)
+			(xy 226.06 54.61) (xy 226.06 53.34)
 		)
 		(stroke
@@
 	(wire
 		(pts
-			(xy 226.06 54.61) (xy 226.06 53.34)
+			(xy 124.46 156.21) (xy 115.57 156.21)
 		)
 		(stroke
@@
 	(wire
 		(pts
-			(xy 125.73 180.34) (xy 125.73 182.88)
+			(xy 30.48 179.07) (xy 30.48 180.34)
 		)
 		(stroke
@@
 	(wire
 		(pts
-			(xy 30.48 179.07) (xy 30.48 180.34)
+			(xy 30.48 162.56) (xy 30.48 165.1)
 		)
 		(stroke
@@
 	(wire
 		(pts
-			(xy 30.48 162.56) (xy 30.48 165.1)
+			(xy 204.47 87.63) (xy 204.47 86.36)
 		)
 		(stroke
@@
 	(wire
 		(pts
-			(xy 204.47 87.63) (xy 204.47 86.36)
+			(xy 215.9 54.61) (xy 226.06 54.61)
 		)
 		(stroke
@@
 	(wire
 		(pts
-			(xy 215.9 54.61) (xy 226.06 54.61)
+			(xy 124.46 167.64) (xy 130.81 167.64)
 		)
 		(stroke
@@
 	(wire
 		(pts
-			(xy 115.57 154.94) (xy 115.57 165.1)
+			(xy 115.57 154.94) (xy 115.57 156.21)
 		)
 		(stroke
@@
 	(wire
 		(pts
-			(xy 125.73 167.64) (xy 125.73 172.72)
-		)
-		(stroke
-			(width 0)
-			(type default)
-		)
-	)
-	(wire
-		(pts
 			(xy 204.47 96.52) (xy 210.82 96.52)
 		)
@@
 	(wire
 		(pts
+			(xy 124.46 158.75) (xy 124.46 156.21)
+		)
+		(stroke
+			(width 0)
+			(type default)
+		)
+	)
+	(wire
+		(pts
 			(xy 207.01 45.72) (xy 207.01 44.45)
 		)
@@
 	(symbol
 		(lib_id "Device:R")
-		(at 125.73 176.53 0)
+		(at 124.46 162.56 0)
 		(unit 1)
 		(body_style 1)
@@
 		(dnp no)
 		(property "Reference" "R51"
-			(at 127.254 175.26 0)
+			(at 125.984 161.29 0)
 			(show_name no)
 			(do_not_autoplace no)
@@
 		)
 		(property "Value" "10k"
-			(at 127.254 177.8 0)
+			(at 125.984 163.83 0)
 			(show_name no)
 			(do_not_autoplace no)
@@
 		)
 		(property "Footprint" "Resistor_SMD:R_0402_1005Metric"
-			(at 123.952 176.53 90)
+			(at 122.682 162.56 90)
 			(hide yes)
 			(show_name no)
@@
 		)
 		(property "Datasheet" ""
-			(at 125.73 176.53 0)
+			(at 124.46 162.56 0)
 			(hide yes)
 			(show_name no)
@@
 		)
 		(property "Description" "Resistor"
-			(at 125.73 176.53 0)
+			(at 124.46 162.56 0)
 			(hide yes)
 			(show_name no)
